File: edge connector breakout/edge connector breakout.kicad_pcb (KiCad board)
At the start: 2 copper layers, 50.8 x 58.4 mm, 3 parts, among them J1 C64 Card Edge, J2 0.1" header

Commit message: breakout: add CC0 to the copyright line
Other:
- board text added: "© 2020 Matt Mullins CC0 No Rights Reserved"
- board text removed: "© 2020 Matt Mullins No Rights Reserved"
Changed lines of the file:
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@@
     )
   )
-  (gr_text "© 2020 Matt Mullins\nNo Rights Reserved" (at 64.008 52.07 90) (layer B.SilkS)
+  (gr_text "© 2020 Matt Mullins\nCC0 No Rights Reserved" (at 64.008 52.07 90) (layer B.SilkS)
     (effects (font (size 1 1) (thickness 0.15)) (justify mirror))
   )
